File: cc1101-sniffer.sch (EAGLE design)
At the start: 39 parts, among them J1 USB4105-GF-A, J2 61300411821, U1 AP2112K, U2 RP2040, U3 W25Q32JVSSIQ, Y1 ABM8G-12.000MHZ-18-D2Y-T3

Commit message: tCream for USB and E01-900M10S
Parts:
- removed U$2: CC1101-868MS10, codm:CC1101-868MS10
- removed U3: W25Q32JVSSIQ, W25Q32JVSSIQ:W25Q32JVSSIQ
- removed X1: (no value), adafruit:ANTENNA_U.FL
- added J3: 61300311821, Eagle_WR-PHD (rev21a):6130XX11821_61300311821
- added R11: 5k1, codm:R-EU_R0603RF
- added U$6: E07-900M10S, codm:E07-900M10S
- added U4: W25Q32JVZPIQ, W25Q32JVZPIQ:W25Q32JVZPIQ
Connections:
- removed net N$5: U$2.ANT, X1.SIGNAL
- new net N$9: J1.CC2, R11.2
- new net SWCLK: J3.1, U2.SWCLK
- new net SWD: J3.3, U2.SWD
- net +3V3: now also U$6.VCC, U4.VCC; no longer U$2.VCC, U3.VCC
- net CSN: now also U$6.CSN, U2.GPIO17; no longer U$2.CSN
- net GDO0: now also U$6.GDO0, U2.GPIO20; no longer U$2.GDO0
- net GND: now also J3.2, R11.1, U$6.GND, U4.GND; no longer U$2.ANTGND, U$2.GND, U3.GND, X1.GND@0, X1.GND@1
- net LED0: now also U2.GPIO25
- net MISO: now also U$6.MISO/GDO1, U2.GPIO16; no longer U$2.MISO
- net MOSI: now also U$6.MOSI, U2.GPIO19; no longer U$2.MOSI
- net QSPI_CSN: now also U4.!CS; no longer U3.!CS
- net QSPI_SCLK: now also U4.CLK; no longer U3.CLK
- net QSPI_SD0: now also U4.DI(IO0); no longer U3.DI(IO0)
- net QSPI_SD1: now also U4.DO(IO1); no longer U3.DO(IO1)
- net QSPI_SD2: now also U4.!WP!(IO2); no longer U3.!WP!(IO2)
- net QSPI_SD3: now also U4.!HOLD/RESET!(IO3); no longer U3.!HOLD!/!RESET!(IO3)
- net SCL: now also U2.GPIO5; no longer U2.GPIO17
- net SCLK: now also U$6.SCK, U2.GPIO18; no longer U$2.SCK
- net SDA: now also U2.GPIO4; no longer U2.GPIO16
Other:
- moved on the sheet: BOOT, C17, C3, C4, C5, D1, J2, R10, R2, R3, R4, R5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
